File: Hardware/Solar_LiPo_charger.kicad_sch (KiCad schematic)
At the start: 77 parts, among them IC1 CN3791, IC2 PAM2423AECADJR, J1 Battery_connector, J2 Solar connectors, J3 Solar connectors, J4 USB_C_Receptacle_USB2.0_16P, J5 Conn_01x02_Pin, J6 5v_out, Q1 PMOS, Q2 NMOS, Q3 NMOS, U2 AP9101CK6

Commit message: Fixed the working of a buck charger for the battery
Parts:
- C14, C21: value 470n -> 10u
- C17, C8: value 22u -> 10u
- C18: value 4.7u -> 10u
- C22: value 10u -> 22u
- C4: value 4.7u -> 22u
- R5: value 470 -> 5k
Connections:
- net GND: now also D4.2 (A)
- net at Q1.1 (D): now also D4.1 (K), L2.1; no longer D4.2 (A)
Other:
- note added: "D+ i D- powinny być połączone telefony sprawdzają linie D+ i D- jeśli nie są połączone to uznają że ładowarka jest najgorszego sortu pobierają najmniejszą ilość prądu"
- note added: "Tu był błąd D4 szło od pmos do cewki Zmieniono na pmos prosto do cewki Wstawiono diode między nie i do masy"
- note added: "Wartość rezystora przed diodami wylicz i wlutuj dopiero jak zobaczysz jakie dostajesz napięcie, na początku 5k"
- moved on the sheet: D4
Changed lines of the file:
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@@
 		)
 	)
+	(text "Tu był błąd D4 szło od pmos do cewki\nZmieniono na pmos prosto do cewki\nWstawiono diode między nie i do masy\n"
+		(exclude_from_sim no)
+		(at 45.72 18.796 0)
+		(effects
+			(font
+				(size 1.27 1.27)
+			)
+		)
+	)
 	(text "Ochrona baterii, powinna działać dla 6A w jedną i drugą stronę"
 		(exclude_from_sim no)
@@
 		)
 	)
+	(text "Wartość rezystora przed diodami wylicz i wlutuj dopiero jak zobaczysz\n jakie dostajesz napięcie, na początku 5k"
+		(exclude_from_sim no)
+		(at 51.308 100.584 0)
+		(effects
+			(font
+				(size 1.27 1.27)
+			)
+		)
+	)
+	(text "D+ i D- powinny być połączone\ntelefony sprawdzają linie D+ i D-\njeśli nie są połączone\nto uznają że ładowarka\njest najgorszego sortu\npobierają najmniejszą\nilość prądu\n"
+		(exclude_from_sim no)
+		(at 125.222 163.83 0)
+		(effects
+			(font
+				(size 1.27 1.27)
+			)
+		)
+	)
 	(junction
 		(at 218.44 116.84)
@@
 	)
 	(junction
+		(at 91.44 29.21)
+		(diameter 0)
+		(color 0 0 0 0)
+	)
+	(junction
 		(at 24.13 59.69)
 		(diameter 0)
@@
 	(wire
 		(pts
+			(xy 74.93 29.21) (xy 91.44 29.21)
+		)
+		(stroke
+			(width 0)
+			(type default)
+		)
+	)
+	(wire
+		(pts
 			(xy 220.98 146.05) (xy 220.98 151.13)
 		)
@@
 	(wire
 		(pts
+			(xy 91.44 29.21) (xy 100.33 29.21)
+		)
+		(stroke
+			(width 0)
+			(type default)
+		)
+	)
+	(wire
+		(pts
 			(xy 248.92 91.44) (xy 248.92 93.98)
 		)
@@
 	(wire
 		(pts
-			(xy 95.25 29.21) (xy 100.33 29.21)
-		)
-		(stroke
-			(width 0)
-			(type default)
-		)
-	)
-	(wire
-		(pts
 			(xy 256.54 104.14) (xy 265.43 104.14)
 		)
@@
 	(wire
 		(pts
-			(xy 74.93 29.21) (xy 87.63 29.21)
-		)
-		(stroke
-			(width 0)
-			(type default)
-		)
-	)
-	(wire
-		(pts
 			(xy 97.79 53.34) (xy 120.65 53.34)
 		)
@@
 		(on_board yes)
 		(dnp no)
-		(fields_autoplaced yes)
 		(property "Reference" "C14"
-			(at 53.34 31.7499 0)
+			(at 48.768 24.638 0)
 			(effects
 				(font
@@
 			)
 		)
-		(property "Value" "470n"
-			(at 53.34 34.2899 0)
+		(property "Value" "10u"
+			(at 49.022 26.924 0)
 			(effects
 				(font
@@
 			)
 		)
-		(property "Value" "10u"
+		(property "Value" "22u"
 			(at 32.766 139.7 0)
 			(effects
@@
 			)
 		)
-		(property "Value" "22u"
+		(property "Value" "10u"
 			(at 99.822 137.922 0)
 			(effects
@@
 			)
 		)
-		(property "Datasheet" "https://ngspice.sourceforge.io/docs/ngspice-html-manual/manual.xhtml#cha_MOSFETs"
+		(property "Datasheet" "https://www.tme.eu/pl/details/ao4407a/tranzystory-z-kanalem-p-smd/alpha-omega-semiconductor/"
 			(at 57.15 31.75 0)
 			(effects
@@
 			)
 		)
-		(property "Datasheet" "https://ngspice.sourceforge.io/docs/ngspice-html-manual/manual.xhtml#cha_MOSFETs"
+		(property "Datasheet" "https://www.tme.eu/pl/details/wms15n03t1-cyg/tranzystory-z-kanalem-n-smd/wayon/wms15n03t1/"
 			(at 264.16 20.32 0)
 			(effects
@@
 	(symbol
 		(lib_id "Diode:SS34")
-		(at 91.44 29.21 180)
+		(at 91.44 33.02 270)
 		(unit 1)
 		(exclude_from_sim no)
@@
 		(fields_autoplaced yes)
 		(property "Reference" "D4"
-			(at 91.7575 22.86 0)
+			(at 93.98 31.4324 90)
 			(effects
 				(font
 					(size 1.27 1.27)
 				)
+				(justify left)
 			)
 		)
 		(property "Value" "SL82-3G"
-			(at 91.7575 25.4 0)
+			(at 93.98 33.9724 90)
 			(effects
 				(font
 					(size 1.27 1.27)
 				)
+				(justify left)
 			)
 		)
 		(property "Footprint" "Diode_SMD:D_SMC"
-			(at 91.44 24.765 0)
+			(at 86.995 33.02 0)
 			(effects
 				(font
@@
 		)
 		(property "Datasheet" "https://www.vishay.com/docs/88751/ss32.pdf"
-			(at 91.44 29.21 0)
+			(at 91.44 33.02 0)
 			(effects
 				(font
@@
 		)
 		(property "Description" "40V 3A Schottky Diode, SMA"
-			(at 91.44 29.21 0)
+			(at 91.44 33.02 0)
 			(effects
 				(font
@@
 			)
 		)
-		(property "Datasheet" "https://www.way-on.cn/upload/202301/31/202301311441465755.pdf"
+		(property "Datasheet" "https://www.tme.eu/pl/details/wms15n03t1-cyg/tranzystory-z-kanalem-n-smd/wayon/wms15n03t1/"
 			(at 264.16 55.88 0)
 			(effects
@@
 			)
 		)
-		(property "Value" "4.7u"
-			(at 109.474 138.938 0)
+		(property "Value" "10u"
+			(at 109.474 138.176 0)
 			(effects
 				(font
@@
 			)
 		)
-		(property "Value" "470"
+		(property "Value" "5k"
 			(at 26.67 57.1499 0)
 			(effects
@@
 			)
 		)
-		(property "Value" "4.7u"
+		(property "Value" "22u"
 			(at 39.116 139.7 0)
 			(effects
@@
 			)
 		)
-		(property "Value" "22u"
+		(property "Value" "10u"
 			(at 104.648 138.176 0)
 			(effects
@@
 	(symbol
 		(lib_id "power:GND")
+		(at 91.44 36.83 0)
+		(unit 1)
+		(exclude_from_sim no)
+		(in_bom yes)
+		(on_board yes)
+		(dnp no)
+		(fields_autoplaced yes)
+		(property "Reference" "#PWR037"
+			(at 91.44 43.18 0)
+			(effects
+				(font
+					(size 1.27 1.27)
+				)
+				(hide yes)
+			)
+		)
+		(property "Value" "GND"
+			(at 91.44 41.91 0)
+			(effects
+				(font
+					(size 1.27 1.27)
+				)
+			)
+		)
+		(property "Footprint" ""
+			(at 91.44 36.83 0)
+			(effects
+				(font
+					(size 1.27 1.27)
+				)
+				(hide yes)
+			)
+		)
+		(property "Datasheet" ""
+			(at 91.44 36.83 0)
+			(effects
+				(font
+					(size 1.27 1.27)
+				)
+				(hide yes)
+			)
+		)
+		(property "Description" "Power symbol creates a global label with name \"GND\" , ground"
+			(at 91.44 36.83 0)
+			(effects
+				(font
+					(size 1.27 1.27)
+				)
+				(hide yes)
+			)
+		)
+		(pin "1"
+		)
+		(instances
+			(project "Solar_LiPo_charger"
+				(path "/929c46f8-95fd-4d35-95df-ed136586ef48"
+					(reference "#PWR037")
+					(unit 1)
+				)
+			)
+		)
+	)
+	(symbol
+		(lib_id "power:GND")
 		(at 129.54 36.83 0)
 		(unit 1)
@@
 			)
 		)
-		(property "Value" "470n"
+		(property "Value" "10u"
 			(at 133.35 26.416 0)
 			(effects
@@
 		(dnp no)
 		(property "Reference" "C19"
-			(at 128.524 24.384 0)
+			(at 127.762 24.13 0)
 			(effects
 				(font
@@
 		)
 		(property "Value" "10u"
-			(at 129.032 27.178 0)
+			(at 128.27 26.416 0)
 			(effects
 				(font
